Commit message: Add files via upload

File: pratica_2/models/my_robot/model.urdf (robot description, URDF)
Before this commit: robot my_robot, 3 links, 2 joints
Links:
- added link caster, mass 0.05; collision sphere radius=0.05; visual sphere radius=0.05
- link chassis: geometry collision box size=0.4 0.2 0.1; visual box size=0.4 0.2 0.1
Joints:
- added joint caster_joint: type fixed, parent chassis, child caster, origin xyz=-0.15 0 -0.05 rpy=0 0 0
- joint left_wheel_hinge: origin xyz=0.1 0.13 0 rpy=0 0 0 -> xyz=0.1 0.13 0.0 rpy=0 0 0
- joint right_wheel_hinge: origin xyz=0.1 -0.13 0 rpy=0 0 0 -> xyz=0.1 -0.13 0.0 rpy=0 0 0

Commit message: Add files via upload

File: pratica_2/models/my_robot/model.urdf (robot description, URDF)
Before this commit: robot my_robot, 4 links, 3 joints
Links:
- removed link caster
- added link caster_link, mass 0.01; collision sphere radius=0.05; visual sphere radius=0.05
- link chassis: geometry collision box size=0.4 0.2 0.1; visual mesh filename=package://pioneer2dx/meshes/chassis.dae scale=0.9 0.5 0.5
Joints:
- joint caster_joint: child caster -> caster_link
- joint left_wheel_hinge: origin xyz=0.1 0.13 0.0 rpy=0 0 0 -> xyz=0.1 0.13 0 rpy=0 0 0
- joint right_wheel_hinge: origin xyz=0.1 -0.13 0.0 rpy=0 0 0 -> xyz=0.1 -0.13 0 rpy=0 0 0
